Commit message: added a lidar link to the model and configured it to work.

File: src/my_robot_description/urdf/mobile_base.xacro (robot description, xacro)
@@ -22,4 +22,23 @@
             </collision>
             <xacro:cylinder_inertia m="1.0" r="${wheel_radius}" l="${wheel_length}" o_xyz="0 0 0" o_rpy="${pi / 2.0} 0 0"/>
+        </link>
+    </xacro:macro>
+    <!-- Added a lidar link macro-->
+    <xacro:macro name="lidar_link" params="suffix">
+        <link name="lidar_${suffix}">
+            <visual>
+                <geometry>
+                    <cylinder radius="${wheel_radius}" length="${wheel_length}" />
+                </geometry>
+                <origin xyz=" 0 0 0 " rpy="0 0 0" />
+                <material name="gray" />
+            </visual>
+            <collision>
+                <geometry>
+                    <cylinder radius="${wheel_radius}" length="${wheel_length}" />
+                </geometry>
+                <origin xyz="0 0 0" rpy="0 0 0" />
+            </collision>
+            <xacro:cylinder_inertia m="1.0" r="${wheel_radius}" l="${wheel_length}" o_xyz="0 0 0" o_rpy="0 0 0"/>
         </link>
     </xacro:macro>
@@ -48,4 +67,5 @@
     <xacro:wheel_link prefix="right" />
     <xacro:wheel_link prefix="left"  />
+    <xacro:lidar_link suffix="0"  />
     <joint name="base_right_wheel_joint" type="continuous">
         <parent link="base_link" />
@@ -58,4 +78,10 @@
         <child link="left_wheel_link" />
         <origin xyz="${-base_length / 4.0} ${(base_width + wheel_length) / 2.0} 0" rpy="0 0 0" />
+        <axis xyz=" 0 1 0 " />
+    </joint>
+    <joint name="base_lidar_joint" type="fixed">
+        <parent link="base_link" />
+        <child link="lidar_0" />
+        <origin xyz="${base_length / 3.0} 0 ${base_height}" rpy="0 0 0" />
         <axis xyz=" 0 1 0 " />
     </joint>

File: src/my_robot_description/urdf/mobile_base_gazebo.xacro (robot description, xacro)
@@ -1,7 +1,43 @@
 <?xml version="1.0"?>
 <robot xmlns:xacro="http://www.ros.org/wiki/xacro">
+    <gazebo>
+        <plugin
+            filename="gz-sim-sensors-system"
+            name="gz::sim::systems::Sensors">
+            <render_engine>ogre2</render_engine>
+        </plugin>
+    </gazebo>
     <gazebo reference="caster_wheel_link">
         <mu1 value="0.1" />
         <mu2 value="0.1" />
+    </gazebo>
+    <gazebo reference="lidar_0">
+        <sensor name="lidar_sensor" type="gpu_lidar">
+            <pose relative_to='lidar_0'>0 0 0 0 0 0</pose>
+            <update_rate>10</update_rate>
+            <topic>scan</topic>
+            <lidar>
+                <scan>
+                    <horizontal>
+                        <samples>720</samples>
+                        <resolution>1</resolution>
+                        <min_angle>-3.14</min_angle>
+                        <max_angle>3.14</max_angle>
+                    </horizontal>
+                </scan>
+                <range>
+                    <min>0.12</min>
+                    <max>10.0</max>
+                    <resolution>0.01</resolution>
+                </range>
+                <noise>
+                    <type>gaussian</type>
+                    <mean>0.0</mean>
+                    <stddev>0.001</stddev>
+                </noise>
+            </lidar>
+            <always_on>1</always_on>
+            <visualize>1</visualize>
+        </sensor>
     </gazebo>
     <gazebo>
